File: FC-v1/FC-v1/FC-v1.kicad_pcb (KiCad board)
At the start: 2 copper layers, 94.4 x 94.4 mm, 16 parts, among them J1 530470610, J2 Left, J3 Right, J4 530470610, U1 ESP32-C3_SUPERMINI_TH

Commit message: CAD files
Parts:
- added G***: LOGO, AutoFly:HCBW, F.Cu at (115.5, 104.8)
- added G***: LOGO, AutoFly:HC, F.Cu at (174.0, 58.8)
